File: Hardware/Project/Project_2_smaller.kicad_pcb (KiCad board)
At the start: 4 copper layers, 95 x 108.9 mm, 80 parts, among them J1 USB_B_Micro, J10 Conn_01x02, J11 Conn_01x02, J12 Conn_01x02, J13 Screen, J14 Conn_01x08_Male, J2 PJ-202-AH, J3 Micro_SD_Card_Det, J5 Conn_01x08_Male, J6 Conn_01x02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

Commit message: update 21-03-21
Parts:
- removed BT1: Battery_Cell, digikey-footprints:Battery_Holder_Coin_2032_BS-7
- removed C1, C12, C4, C5: 1n, Capacitor_SMD:C_0402_1005Metric
- removed C10, C14, C8: 4u7, Capacitor_SMD:C_0402_1005Metric
- removed C11, C13, C15, C2, C3, C6, C7, C9: 100n, Capacitor_SMD:C_0402_1005Metric
- removed C16, C17, C18: 10n, Capacitor_SMD:C_0402_1005Metric
- removed D1, D2: PSM712-LF-T7, Package_TO_SOT_SMD:SOT-23
- removed J1: USB_B_Micro, digikey-footprints:USB_Micro_B_Female_10118194-0001LF
- removed J10, J11, J12, J6, J7, J8, J9: Conn_01x02, Connector_PinHeader_2.54mm:PinHeader_1x02_P2.54mm_Vertical
- removed J13: Screen, Connector_PinSocket_2.54mm:PinSocket_1x05_P2.54mm_Vertical
- removed J2: PJ-202-AH, digikey-footprints:Barrel_Jack_5.5mmODx2.1mmID_PJ-202A
- removed J3: Micro_SD_Card_Det, digikey-footprints:GCT_MEM2075-00-140-01-A
- removed J5: Conn_01x08_Male, Connector_PinHeader_2.54mm:PinHeader_1x08_P2.54mm_Vertical
- removed Q1, Q2: MMBT3904, Package_TO_SOT_SMD:SOT-23
- removed R1, R10, R11, R2, R3, R4, R5, R6, R7, R8, R9: 10k, Resistor_SMD:R_0603_1608Metric
- removed REF** (x2): MountingHole_2.2mm_M2, MountingHole:MountingHole_2.2mm_M2
- removed S1: PEC11R-4020F-S0024, digikey-footprints:Rotary_Encoder_Switched_PEC11R
- removed SW1: RESET, digikey-footprints:Switch_Tactile_SMD_4.5x4.5mm_TL3315NF160Q
- removed U1: ESP32-WROOM-32, RF_Module:ESP32-WROOM-32
- removed U2: LM7812_TO220, Package_TO_SOT_THT:TO-220-3_Horizontal_TabDown
- removed U3: DS3231M, Package_SO:SOIC-16W_7.5x10.3mm_P1.27mm
- removed U4: CP2104, Package_DFN_QFN:QFN-24-1EP_4x4mm_P0.5mm_EP2.6x2.6mm
- removed U5: AMS1117-3.3, Package_TO_SOT_SMD:SOT-223-3_TabPin2
Connections:
- D10 pad 1: Net-(D10-Pad1) -> Earth
- D14 pad 1: Net-(D12-Pad1) -> Earth
- D17 pad 1: Net-(D15-Pad1) -> Earth
- D20 pad 1: Net-(D18-Pad1) -> Earth
- D5 pad 1: Net-(D3-Pad1) -> Earth
- D7 pad 1: Net-(D6-Pad1) -> Earth
- Q3 pad 2: Earth -> Net-(Q3-Pad2)
- Q3 pad 3: Net-(D3-Pad1) -> +12V
- Q4 pad 2: Earth -> Net-(Q4-Pad2)
- Q4 pad 3: Net-(D6-Pad1) -> +12V
- Q5 pad 2: Earth -> Net-(Q5-Pad2)
- Q5 pad 3: Net-(D10-Pad1) -> +12V
- Q6 pad 2: Earth -> Net-(Q6-Pad2)
- Q6 pad 3: Net-(D12-Pad1) -> +12V
- Q7 pad 2: Earth -> Net-(Q7-Pad2)
- Q7 pad 3: Net-(D15-Pad1) -> +12V
- Q8 pad 2: Earth -> Net-(Q8-Pad2)
- Q8 pad 3: Net-(D18-Pad1) -> +12V
- R18 pad 2: +12V -> Net-(Q3-Pad2)
- R19 pad 2: +12V -> Net-(Q4-Pad2)
- R20 pad 2: +12V -> Net-(Q5-Pad2)
- R21 pad 2: +12V -> Net-(Q6-Pad2)
- R22 pad 2: +12V -> Net-(Q7-Pad2)
- R23 pad 2: +12V -> Net-(Q8-Pad2)
Routing:
- net Net-(D18-Pad1): track 68.5 -> 0.00 mm
- net Net-(Q8-Pad2): track 0.00 -> 63.4 mm
- net +3V3: track 59.3 -> 0.00 mm, vias 8 -> 0
- net /PWM6: track 66.2 -> 9.52 mm, vias 1 -> 0
- net SDA: track 55.9 -> 0.00 mm, vias 1 -> 0
- net SCL: track 54.3 -> 0.00 mm
- net /PWM5: track 60.4 -> 6.50 mm, vias 1 -> 0
- net Earth: track 53.1 -> 0.00 mm, vias 14 -> 1
- net /PWM3: track 53.4 -> 3.63 mm, vias 1 -> 0
- net /PWM4: track 51.8 -> 3.48 mm, vias 1 -> 0
- net /OnOff: track 46.8 -> 0.00 mm
- net /PWM2: track 51.3 -> 6.62 mm, vias 1 -> 0
- net /PWM1: track 51.6 -> 9.76 mm, vias 1 -> 0
- net Net-(D15-Pad1): track 41.5 -> 0.00 mm
- net /RTC-INTSQW: track 36.9 -> 0.00 mm, vias 2 -> 0
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Other:
- board size 95 x 108.9 mm -> 43 x 56.7 mm
